Commit message: modified accesories.urdf.xacro to account for kinect2. Don't think it will work as-is. Going to try just referencing kinect2 file at launch

File: jpbos/jackal_description/urdf/accessories.urdf.xacro (robot description, xacro)
@@ -25,4 +25,16 @@
       <parent link="$(optenv JACKAL_LASER_MOUNT front)_mount" />
       <child link="$(optenv JACKAL_LASER_MOUNT front)_laser_mount" />
+    </joint>
+  </xacro:if>
+<!-- If enabled, generate the Kinect2 payload  -->
+  <xacro:include filename="accessories/kinect2.urdf.xacro" />
+  <xacro:if value="$(optenv KINECT2 0)">
+    <sick_lms1xx_mount prefix="$(optenv JACKAL_KINECT2_MOUNT front)"
+                       topic="$(optenv JACKAL_KINECT2_TOPIC front/scan)"/>
+    <joint name="$(optenv JACKAL_KINECT2_MOUNT front)_kinect2_mount_joint" type="fixed">
+      <origin xyz="$(optenv JACKAL_KINECT2_OFFSET 0 0 0)"
+              rpy="$(optenv JACKAL_KINECT2_RPY 0 0 0)" />
+      <parent link="$(optenv JACKAL_KINECT2_MOUNT front)_mount" />
+      <child link="$(optenv JACKAL_KINECT2_MOUNT front)_laser_mount" />
     </joint>
   </xacro:if>
